File: Hardware/CitizenBoard V3.2.brd (EAGLE design)
At the start: 50 x 50 mm, 28 parts, among them IC1 MEGA8-P, J1 DCJ0202, J2 AUDIO-JACK-3.5, Y1 16MHz

Commit message: v1.0 sent for printing, after minor update
Parts:
- added C4: 0.1 µF 6V, rcl:C025-024X044
- added JP5: (no value), pinhead:1X04
- C5: value 0.1 µF 6V -> 10uF; device rcl:C025-024X044 -> rcl:E2,5-6E
- J1: device con-jack:DCJ0202 -> con-jack_modified:DCJ0202
- moved LED1 15.3 mm to (2.54, 31.8)
- moved Y1 8.89 mm to (44.5, 2.54)
- moved LED2 8.52 mm to (7.62, 31.8)
- moved C5 8.52 mm to (6.35, 11.4), turned to 180 degrees
- moved R12 8.03 mm to (15.2, 29.2)
- moved FTDI 7.62 mm to (27.9, 2.54)
- moved R5 6.35 mm to (10.2, 6.35), turned to 90 degrees
- moved R8 5.68 mm to (15.2, 31.8)
- moved JP1 4.02 mm to (24.1, 36.8), turned to 90 degrees
- moved C3 2.84 mm to (17.8, 35.6)
- moved J2 1.27 mm to (7.62, 44.5)
- moved R1 1.27 mm to (19.1, 45.7)
- moved R2 1.27 mm to (19.1, 40.6)
- moved R3 1.27 mm to (19.1, 43.2)
- moved R4 1.27 mm to (22.9, 26.7)
Connections:
- new net SHND: JP5.1
- new net VIN: JP4.2, JP5.2
- net GND: now also C5.-, JP5.3
- net N$3: now also C4.1; no longer C5.1
- net RESET: now also C4.2; no longer C5.2
- net VCC: now also C5.+, JP5.4; no longer JP4.2
Routing:
- net VIN: track 0.00 -> 15.7 mm
- net D2: track 25.4 -> 35.2 mm, vias 1 -> 0
- net TOSC2: track 9.42 -> 16.8 mm
- net RX: track 9.94 -> 16.8 mm
- net N: track 29.3 -> 35.0 mm
- net TOSC1: track 9.42 -> 14.3 mm
- net VCC: track 94.4 -> 98.5 mm, vias 2 -> 0
- net N$4: track 23.2 -> 19.9 mm
- net N$5: track 12.5 -> 10.5 mm
- net ADC0: track 8.89 -> 7.62 mm
- net RESET: track 14.0 -> 12.7 mm
- net N$3: track 3.81 -> 5.08 mm
- net TX: track 9.94 -> 11.0 mm
- net N$2: track 6.35 -> 5.39 mm
- net D3: track 31.8 -> 32.7 mm, vias 2 -> 0
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Other:
- board text added: "/home/phyks/hackEns/CitizenWatt/CitizenWatt-sensor/Hardware/silkscreen3bold.bmp"
- board text added: "1"
- board text added: "CitizenBoard v1.0"
- board text added: "VOUT"
- board text removed: "/home/phyks/hackEns/CitizenWatt/CitizenWatt-sensor/Hardware/CitizenBoard/silkscreen3bold.bmp"
