File: Hardware/CitizenBoard V3.2.sch (EAGLE design)
At the start: 28 parts, among them IC1 MEGA8-P, J1 DCJ0202, J2 AUDIO-JACK-3.5, Y1 16MHz

Commit message: v1.0 sent for printing, after minor update
Parts:
- added C4: 0.1 µF 6V, rcl:C-EU025-024X044
- added JP5: (no value), pinhead:PINHD-1X4
- C5: value 0.1 µF 6V -> 10uF; device rcl:C-EU025-024X044 -> rcl:CPOL-EUE2,5-6E
- J1: device con-jack:DCJ0202 -> con-jack_modified:DCJ0202
Connections:
- new net SHND: JP5.1
- new net VIN: JP4.2, JP5.2
- net GND: now also C5.-, JP5.3
- net N$3: now also C4.1; no longer C5.1
- net RESET: now also C4.2; no longer C5.2
- net VCC: now also C5.+, JP5.4; no longer JP4.2
Changed lines of the file:
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@@
 <part name="JP1" library="pinhead" deviceset="PINHD-1X2" device=""/>
 <part name="R4" library="rcl" deviceset="R-EU_" device="0204/7" value="1K"/>
-<part name="C5" library="rcl" deviceset="C-EU" device="025-024X044" value="0.1 µF 6V"/>
+<part name="C4" library="rcl" deviceset="C-EU" device="025-024X044" value="0.1 µF 6V"/>
 <part name="R5" library="rcl" deviceset="R-EU_" device="0204/7" value="10K"/>
-<part name="J1" library="con-jack" deviceset="DCJ0202" device=""/>
+<part name="J1" library="con-jack_modified" deviceset="DCJ0202" device=""/>
 <part name="JP2" library="pinhead" deviceset="PINHD-1X14" device=""/>
 <part name="JP3" library="pinhead" deviceset="PINHD-1X14" device=""/>
@@
 <part name="P+2" library="supply1" deviceset="VCC" device=""/>
 <part name="J2" library="alex" deviceset="AUDIO-JACK-3.5" device=""/>
+<part name="P+3" library="supply1" deviceset="VCC" device=""/>
+<part name="GND5" library="supply1" deviceset="GND" device=""/>
+<part name="C5" library="rcl" deviceset="CPOL-EU" device="E2,5-6E" value="10uF"/>
+<part name="JP5" library="pinhead" deviceset="PINHD-1X4" device=""/>
 </parts>
 <sheets>
@@
 <instance part="JP1" gate="G$1" x="63.5" y="109.22"/>
 <instance part="R4" gate="G$1" x="40.64" y="119.38" rot="R90"/>
-<instance part="C5" gate="G$1" x="17.78" y="58.42" rot="R90"/>
+<instance part="C4" gate="G$1" x="17.78" y="58.42" rot="R90"/>
 <instance part="R5" gate="G$1" x="27.94" y="63.5" rot="R90"/>
 <instance part="J1" gate="G$1" x="99.06" y="91.44"/>
@@
 <instance part="P+2" gate="VCC" x="27.94" y="76.2"/>
 <instance part="J2" gate="G$1" x="12.7" y="104.14"/>
+<instance part="P+3" gate="VCC" x="198.12" y="53.34"/>
+<instance part="GND5" gate="1" x="198.12" y="35.56"/>
+<instance part="C5" gate="G$1" x="198.12" y="45.72"/>
+<instance part="JP5" gate="A" x="172.72" y="43.18"/>
 </instances>
 <busses>
@@
 </segment>
 <segment>
-<pinref part="JP4" gate="G$1" pin="1"/>
-<wire x1="160.02" y1="43.18" x2="154.94" y2="43.18" width="0.1524" layer="91"/>
-<junction x="154.94" y="43.18"/>
-<label x="160.02" y="43.18" size="1.778" layer="95"/>
-</segment>
-<segment>
 <pinref part="IC1" gate="G$1" pin="GND"/>
 <wire x1="50.8" y1="53.34" x2="45.72" y2="53.34" width="0.1524" layer="91"/>
@@
 <label x="45.72" y="27.94" size="1.778" layer="95"/>
 </segment>
+<segment>
+<pinref part="JP4" gate="G$1" pin="1"/>
+<wire x1="154.94" y1="43.18" x2="170.18" y2="43.18" width="0.1524" layer="91"/>
+<label x="160.02" y="43.18" size="1.778" layer="95"/>
+<junction x="154.94" y="43.18"/>
+<pinref part="JP5" gate="A" pin="3"/>
+<junction x="170.18" y="43.18"/>
+</segment>
+<segment>
+<pinref part="GND5" gate="1" pin="GND"/>
+<pinref part="C5" gate="G$1" pin="-"/>
+<wire x1="198.12" y1="38.1" x2="198.12" y2="40.64" width="0.1524" layer="91"/>
+<junction x="198.12" y="40.64"/>
+<junction x="198.12" y="38.1"/>
+</segment>
 </net>
 <net name="VCC" class="0">
@@
 <label x="175.26" y="78.74" size="1.778" layer="95"/>
 <junction x="165.1" y="78.74"/>
-</segment>
-<segment>
-<pinref part="JP4" gate="G$1" pin="2"/>
-<wire x1="154.94" y1="45.72" x2="160.02" y2="45.72" width="0.1524" layer="91"/>
-<label x="160.02" y="45.72" size="1.778" layer="95"/>
-<junction x="154.94" y="45.72"/>
 </segment>
 <segment>
@@
 <label x="45.72" y="48.26" size="1.778" layer="95"/>
 </segment>
+<segment>
+<wire x1="170.18" y1="40.64" x2="160.02" y2="40.64" width="0.1524" layer="91"/>
+<label x="160.02" y="40.64" size="1.778" layer="95"/>
+<pinref part="JP5" gate="A" pin="4"/>
+<junction x="170.18" y="40.64"/>
+</segment>
+<segment>
+<pinref part="C5" gate="G$1" pin="+"/>
+<pinref part="P+3" gate="VCC" pin="VCC"/>
+<wire x1="198.12" y1="48.26" x2="198.12" y2="50.8" width="0.1524" layer="91"/>
+<junction x="198.12" y="48.26"/>
+<junction x="198.12" y="50.8"/>
+</segment>
 </net>
 <net name="RX" class="0">
@@
 <junction x="50.8" y="58.42"/>
 <wire x1="50.8" y1="58.42" x2="27.94" y2="58.42" width="0.1524" layer="91"/>
-<pinref part="C5" gate="G$1" pin="2"/>
+<pinref part="C4" gate="G$1" pin="2"/>
 <pinref part="R5" gate="G$1" pin="1"/>
 <junction x="22.86" y="58.42"/>
@@
 <net name="N$3" class="0">
 <segment>
-<pinref part="C5" gate="G$1" pin="1"/>
+<pinref part="C4" gate="G$1" pin="1"/>
 <wire x1="5.08" y1="58.42" x2="15.24" y2="58.42" width="0.1524" layer="91"/>
 <junction x="15.24" y="58.42"/>
@@
 </segment>
 </net>
+<net name="VIN" class="0">
+<segment>
+<pinref part="JP4" gate="G$1" pin="2"/>
+<wire x1="154.94" y1="45.72" x2="170.18" y2="45.72" width="0.1524" layer="91"/>
+<label x="160.02" y="45.72" size="1.778" layer="95"/>
+<junction x="154.94" y="45.72"/>
+<pinref part="JP5" gate="A" pin="2"/>
+<junction x="170.18" y="45.72"/>
+</segment>
+</net>
+<net name="SHND" class="0">
+<segment>
+<pinref part="JP5" gate="A" pin="1"/>
+<wire x1="170.18" y1="48.26" x2="160.02" y2="48.26" width="0.1524" layer="91"/>
+<label x="160.02" y="48.26" size="1.778" layer="95"/>
+<junction x="170.18" y="48.26"/>
+</segment>
+</net>
